File: Hardware/Resnik.sch (EAGLE design)
At the start: 187 parts, among them IC1 ATMEGA644M, J1 CONN_82.54_SCREW, J3 CONN_42.54_SCREW, J4 CONN_82.54_SCREW, Q1 DMG3404, Q2 DMG3404, Q3 FDN360P, Q4 FDN360P, Q5 FDN360P, Q6 DMG3404, U1 TLV61220DBV, U10 TPS22917DBV, U11 SN74AUP1G04YFP, U12 SN74AUP1G04YFP, U13 SN74AUP2G86SOT833-1, U14 SN74AUP2G08DQE, U15 SN74AUP2G08DQE, U16 SN74AUP2G08DQE, U17 MIC2544MSOP, U18 MIC2544MSOP, U19 MIC2544MSOP, U2 TPS62822DLC, U20 MIC2544MSOP, U21 TPS22917DBV, U22 TPS22917DBV, U23 FT231X-Q, U24 SN74LVC1G3157DRL, U25 SN74AUP3G34DCU, U26 TXS0102DQM, U27 TXS0108RGY, U28 TXS0108RGY, U29 TXS0104RGY, U3 TPS61032RSA, U30 MCP4726A2SOT-23, U31 BME280, U32 ADS1115, U33 ADS1115, U34 INA211DCK, U35 INA210DCK, U36 TCA9535RTW, U5 BQ2980RUG, U6 TPS2105, U7 LTC4412S6, U8 TPL5111DDC, U9 TPS79733

Commit message: Initial schematic updated for v0.2
First round of updates to schematic for v0.2 update, needs verification before layout begins
Parts:
- added C43: 100uF, bschulz_passives:CTANT_EU2917
- added JP8: JUMPER-SMT_3_1-NC_PASTE_SILK, SparkFun-Jumpers:JUMPER-SMT_3_1-NC_PASTE_SILK
- added Q7: 2N7002, bschulz:MOSFET-NCH-2N7002PW
- added Q8: FDN360P, bschulz:MOSFET_PCH-FDN360P
- added R62: 330k, bschulz_passives:R-EU_330KR0603
- added R63: 10M, bschulz_passives:R-EU_10MR0603
- added R64: 130k, bschulz_passives:R-EU_130KR0603
- added S5: BUTTON2.6X1.6, bschulz:BUTTON2.6X1.6
- added U$1: MIC94090C6, bschulz:MIC94090C6
- added U37: TLV3691DCK, bschulz:TLV3691DCK
- added U38: TS5A21366DCU, bschulz:TS5A21366DCU
- C15, C16: value 0.1uF -> 0.22uF; device bschulz_passives:C-EU0.1UFC0402 -> bschulz_passives:C-EU0.22UFC0402
- J5, J6, J7: device bschulz:CONN_02SCREW_2.54 -> bschulz:CONN_022.54_SCREW
- R20: value 120k -> 130k; device bschulz_passives:R-EU_120KR0402 -> bschulz_passives:R-EU_130KR0603
Connections:
- new net 3V3_CORE_ISO: C26.1, C27.1, C28.1, R46.2, R47.2, R57.2, R61.2, U$1.VOUT, U26.EN, U26.VA, U27.VA, U28.VA, U29.VA
- new net N$17: Q7.D, Q8.G, R63.2
- new net N$19: JP8.3, R20.1
- new net N$42: JP8.1, R62.1
- new net V_CORE_SW: U37.OUT, U6.EN
- new net V_LI_SENSE: U32.AIN0, U38.B1
- new net V_PRIME_SENSE: Q8.D, U32.AIN2, U38.B2
- net 3V3_AUX: now also U$1.EN; no longer C26.1, C27.1, C28.1, R41.2, R46.2, R47.2, R57.2, R61.2, U26.EN, U26.VA, U27.VA, U28.VA, U29.VA
- net 3V3_CORE: now also R41.2, U$1.VIN
- net 5V_AUX: now also Q7.G, R64.2, U38.S1, U38.S2, U38.VCC
- net 5V_LP: now also U37.IN+; no longer U6.EN
- net GND: now also C43.-, JP8.2, Q7.S, R64.1, U$1.GND, U37.GND, U38.GND; no longer R20.1
- net LI+: now also S5.1, S5.2, U38.A1; no longer U32.AIN0
- net N$63: now also R62.2
- net V_CORE: now also C43.+, U37.VCC
- net V_HP: no longer U21.QOD, U22.QOD
- net V_LI: now also S5.3, S5.4
- net V_PRIME: now also Q8.S, R63.1, U37.IN-, U38.A2; no longer U32.AIN2
Other:
- note added: "Change package???"
- note added: "DELETE!!!!!!"
- note added: "Manual start switch"
- moved on the sheet: C17, C18, U9
