File: Hardware/Okapi.sch (EAGLE design)
At the start: 247 parts, among them IC1 ATMEGA1284M, J1 CONN_82.54_SCREW, J3 CONN_42.54_SCREW, J4 CONN_82.54_SCREW, J9 B_SERIES_M.2EKEY_NOPROG, Q1 DMG3404, Q2 DMG3404, Q3 FDN360P, Q4 2N7002, Q5 FDN360P, Q6 DMG3404, Q7 2N7002, Q8 2N7002, U1 TLV61220DBV, U10 TPS22917DBV, U11 SN74AUP1G04YFP, U12 SN74AUP1G04YFP, U13 SN74AUP1G04YFP, U14 SN74AUP2G08DQE, U15 SN74AUP2G08DQE, U16 SN74AUP2G08DQE, U17 MIC2544MSOP, U18 MIC2544MSOP, U19 MIC2544MSOP, U2 TPS62822DLC, U20 MIC2544MSOP, U21 TPS22917DBV, U22 TPS22917DBV, U23 FT231X-Q, U24 SN74LVC1G3157DRL, U25 SN74AUP3G34DCU, U26 TXS0102DQM, U27 TXS0104RGY, U28 TCA9406DCU, U29 TXS0104RGY, U3 TPS61032RSA, U30 MCP4726A2SOT-23, U31 BME280, U32 PAC1934QFN, U33 ADS1115, U34 TXS0102DQM, U35 MB85RC, U36 TCA9406DCU, U37 TLV3691DCK, U38 MLX90393, U39 MIC94094C6, U40 SN74AHC1G86DCK, U41 MCP23018QFN, U42 TXS0104RGY, U43 BMA456, U44 VEML6030, U45 PCA9634QFN, U5 BQ2980RUG, U6 TPS2105, U7 LTC4412S6, U8 TPL5111DDC, U9 TPS79733

Commit message: v1.0 updates
Parts:
- added R86, R87: (no value), bschulz_passives:R-EU_10KR0402
- added S6, S7: BUTTON4.2X3.2, bschulz:BUTTON4.2X3.2
Connections:
- new net !MODE: J9.MODE, R87.1, S6.1, S6.2
- new net !RST: J9.RESET, R86.1, S7.1, S7.2
- net 3V3_FEATHER: now also R86.2, R87.2
- net GND: now also S6.3, S6.4, S7.3, S7.4
Changed lines of the file:
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@@
 <part name="F2" library="bschulz" deviceset="PPTC" device="1.5A"/>
 <part name="USB2" library="bschulz" deviceset="USB_MICRO" device="VERT"/>
+<part name="S6" library="bschulz" deviceset="BUTTON" device="4.2X3.2"/>
+<part name="S7" library="bschulz" deviceset="BUTTON" device="4.2X3.2"/>
+<part name="R86" library="bschulz_passives" deviceset="R-EU_" device="R0402" technology="10K"/>
+<part name="R87" library="bschulz_passives" deviceset="R-EU_" device="R0402" technology="10K"/>
+<part name="GND104" library="supply1" library_urn="urn:adsk.eagle:library:371" deviceset="GND" device=""/>
+<part name="GND105" library="supply1" library_urn="urn:adsk.eagle:library:371" deviceset="GND" device=""/>
 </parts>
 <sheets>
@@
 <attribute name="VALUE" x="60.96" y="218.44" size="1.27" layer="96"/>
 </instance>
+<instance part="S6" gate="G$1" x="106.68" y="279.4" smashed="yes"/>
+<instance part="S7" gate="G$1" x="106.68" y="259.08" smashed="yes"/>
+<instance part="R86" gate="G$1" x="96.52" y="264.16" smashed="yes" rot="R90">
+<attribute name="NAME" x="95.0214" y="260.35" size="1.778" layer="95" rot="R90"/>
+<attribute name="VALUE" x="99.822" y="260.35" size="1.778" layer="96" rot="R90"/>
+</instance>
+<instance part="R87" gate="G$1" x="96.52" y="284.48" smashed="yes" rot="R90">
+<attribute name="NAME" x="95.0214" y="280.67" size="1.778" layer="95" rot="R90"/>
+<attribute name="VALUE" x="99.822" y="280.67" size="1.778" layer="96" rot="R90"/>
+</instance>
+<instance part="GND104" gate="1" x="127" y="274.32" smashed="yes">
+<attribute name="VALUE" x="124.46" y="271.78" size="1.778" layer="96"/>
+</instance>
+<instance part="GND105" gate="1" x="127" y="254" smashed="yes">
+<attribute name="VALUE" x="124.46" y="251.46" size="1.778" layer="96"/>
+</instance>
 </instances>
 <busses>
@@
 <label x="83.82" y="226.06" size="0.8128" layer="95" xref="yes"/>
 </segment>
+<segment>
+<pinref part="S6" gate="G$1" pin="4"/>
+<pinref part="S6" gate="G$1" pin="3"/>
+<wire x1="121.92" y1="276.86" x2="121.92" y2="279.4" width="0.1524" layer="91"/>
+<junction x="121.92" y="279.4"/>
+<wire x1="121.92" y1="279.4" x2="127" y2="279.4" width="0.1524" layer="91"/>
+<wire x1="127" y1="279.4" x2="127" y2="276.86" width="0.1524" layer="91"/>
+<pinref part="GND104" gate="1" pin="GND"/>
+</segment>
+<segment>
+<pinref part="S7" gate="G$1" pin="4"/>
+<pinref part="S7" gate="G$1" pin="3"/>
+<wire x1="121.92" y1="256.54" x2="121.92" y2="259.08" width="0.1524" layer="91"/>
+<junction x="121.92" y="259.08"/>
+<wire x1="121.92" y1="259.08" x2="127" y2="259.08" width="0.1524" layer="91"/>
+<wire x1="127" y1="259.08" x2="127" y2="256.54" width="0.1524" layer="91"/>
+<pinref part="GND105" gate="1" pin="GND"/>
+</segment>
 </net>
 <net name="MISO" class="0">
@@
 <label x="154.94" y="231.14" size="0.8128" layer="95" xref="yes"/>
 </segment>
+<segment>
+<pinref part="R87" gate="G$1" pin="2"/>
+<wire x1="96.52" y1="289.56" x2="96.52" y2="292.1" width="0.1524" layer="91"/>
+<wire x1="96.52" y1="292.1" x2="91.44" y2="292.1" width="0.1524" layer="91"/>
+<label x="91.44" y="292.1" size="0.8128" layer="95" rot="R180" xref="yes"/>
+</segment>
+<segment>
+<pinref part="R86" gate="G$1" pin="2"/>
+<wire x1="96.52" y1="269.24" x2="96.52" y2="271.78" width="0.1524" layer="91"/>
+<wire x1="96.52" y1="271.78" x2="91.44" y2="271.78" width="0.1524" layer="91"/>
+<label x="91.44" y="271.78" size="0.8128" layer="95" rot="R180" xref="yes"/>
+</segment>
 </net>
 <net name="SCL_FEATHER" class="0">
@@
 </segment>
 </net>
+<net name="!RST" class="0">
+<segment>
+<pinref part="S7" gate="G$1" pin="1"/>
+<pinref part="S7" gate="G$1" pin="2"/>
+<wire x1="106.68" y1="259.08" x2="106.68" y2="256.54" width="0.1524" layer="91"/>
+<junction x="106.68" y="259.08"/>
+<pinref part="R86" gate="G$1" pin="1"/>
+<wire x1="96.52" y1="259.08" x2="106.68" y2="259.08" width="0.1524" layer="91"/>
+<wire x1="96.52" y1="259.08" x2="91.44" y2="259.08" width="0.1524" layer="91"/>
+<junction x="96.52" y="259.08"/>
+<label x="91.44" y="259.08" size="0.8128" layer="95" rot="R180" xref="yes"/>
+</segment>
+<segment>
+<pinref part="J9" gate="U1" pin="RESET"/>
+<wire x1="152.4" y1="200.66" x2="154.94" y2="200.66" width="0.1524" layer="91"/>
+<label x="154.94" y="200.66" size="0.8128" layer="95" xref="yes"/>
+</segment>
+</net>
+<net name="!MODE" class="0">
+<segment>
+<pinref part="S6" gate="G$1" pin="1"/>
+<pinref part="S6" gate="G$1" pin="2"/>
+<wire x1="106.68" y1="279.4" x2="106.68" y2="276.86" width="0.1524" layer="91"/>
+<junction x="106.68" y="279.4"/>
+<pinref part="R87" gate="G$1" pin="1"/>
+<wire x1="106.68" y1="279.4" x2="96.52" y2="279.4" width="0.1524" layer="91"/>
+<wire x1="96.52" y1="279.4" x2="91.44" y2="279.4" width="0.1524" layer="91"/>
+<junction x="96.52" y="279.4"/>
+<label x="91.44" y="279.4" size="0.8128" layer="95" rot="R180" xref="yes"/>
+</segment>
+<segment>
+<pinref part="J9" gate="U1" pin="MODE"/>
+<wire x1="152.4" y1="203.2" x2="154.94" y2="203.2" width="0.1524" layer="91"/>
+<label x="154.94" y="203.2" size="0.8128" layer="95" xref="yes"/>
+</segment>
+</net>
