File: Hardware/KiCAD-10import/Okapi.kicad_sch (KiCad schematic)
At the start: 80 parts, among them Q1 DMG3404, Q2 DMG3404, Q3 FDN360P, Q5 FDN360P, Q6 DMG3404, Q7 2N7002, Q8 2N7002, U1 TLV61220DBV, U10 TPS22917DBV, U13 SN74AUP1G04YFP, U2 TPS6282DLC, U3 TPS61032RSA, U37 TLV3691DCK, U39 MIC94094C6, U4 LT3652DD, U5 BQ2980RUG, U6 TPS2105, U7 LTC4412S6, U8 TPL5111DDC, U9 TPS797

Commit message: KiCAD-10import: fix power net and label errors from Eagle import
- Okapi_2: P+1-4,6-9 → 3V3_AUX; P+5,P+10 → 3V3_CORE (were all VCC)
- Okapi_3: SUPPLY9,SUPPLY10 → 3V3_CORE (were VCC)
- Okapi_5: P+11 → 3V3_AUX (was VCC)
- Okapi_2: QOD global labels → FEATHER_BAT (Eagle net name)
- Okapi root: add V_CORE net label on U6-OUT/U9-VIN/C17/C43 wire

The Eagle→KiCad importer assigns all P+/SUPPLY power symbols the
generic "VCC" net regardless of the actual net they sit on in Eagle.
The correct rail assignments were traced from the Eagle netlist.

Co-Authored-By: Claude Sonnet 4.6 <noreply@anthropic.com>
Connections:
- net V_CORE: now reaches C17.1, C43.+, U6.4 (OUT), U9.4 (VIN)
Changed lines of the file:
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@@
+		)
+	)
+	(label "V_CORE"
+		(at 353.06 55.88 0)
+		(effects
+			(font
+				(size 0.889 0.889)
+			)
+			(justify left bottom)
 		)
 	)
