File: Hardware/KiCAD-10import/Okapi_2.kicad_sch (KiCad schematic)
At the start: 53 parts, among them J10 USB_C, U11 SN74AUP1G04YFP, U12 SN74AUP1G04YFP, U14 SN74AUP2G08DQE, U15 SN74AUP2G08DQE, U16 SN74AUP2G08DQE, U17 MIC2544MSOP, U18 MIC2544MSOP, U19 MIC2544MSOP, U20 MIC2544MSOP, U21 TPS22917DBV, U22 TPS22917DBV, U23 FT231X-Q, U40 SN74AHC1G86DCK

Commit message: KiCAD-10import: fix power net and label errors from Eagle import
- Okapi_2: P+1-4,6-9 → 3V3_AUX; P+5,P+10 → 3V3_CORE (were all VCC)
- Okapi_3: SUPPLY9,SUPPLY10 → 3V3_CORE (were VCC)
- Okapi_5: P+11 → 3V3_AUX (was VCC)
- Okapi_2: QOD global labels → FEATHER_BAT (Eagle net name)
- Okapi root: add V_CORE net label on U6-OUT/U9-VIN/C17/C43 wire

The Eagle→KiCad importer assigns all P+/SUPPLY power symbols the
generic "VCC" net regardless of the actual net they sit on in Eagle.
The correct rail assignments were traced from the Eagle netlist.

Co-Authored-By: Claude Sonnet 4.6 <noreply@anthropic.com>
Connections:
- net 3V3_AUX: now also R24.2, R25.2, S1.1 (O), S2.1 (O), U11.A2 (VCC), U12.A2 (VCC), U14.8 (VCC), U15.8 (VCC)
- net 3V3_CORE: now also U16.8 (VCC), U40.5 (VCC)
- net QOD renamed FEATHER_BAT
- removed net VCC: R24.2, R25.2, S1.1 (O), S2.1 (O), U11.A2 (VCC), U12.A2 (VCC), U14.8 (VCC), U15.8 (VCC), U16.8 (VCC), U40.5 (VCC)
Changed lines of the file:
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@@
 		)
 	)
-	(global_label "QOD"
+	(global_label "FEATHER_BAT"
 		(shape bidirectional)
 		(at 132.08 180.34 0)
@@
 		)
 	)
-	(global_label "QOD"
+	(global_label "FEATHER_BAT"
 		(shape bidirectional)
 		(at 132.08 203.2 0)
@@
 	)
 	(symbol
-		(lib_id "Okapi-eagle-import:supply1_371_VCC")
+		(lib_id "Okapi-eagle-import:3V3_CORE")
 		(at 78.74 175.26 0)
 		(unit 1)
@@
 			)
 		)
-		(property "Value" "VCC"
+		(property "Value" "3V3_CORE"
 			(at 76.2 177.8 90)
 			(show_name no)
@@
 	)
 	(symbol
-		(lib_id "Okapi-eagle-import:supply1_371_VCC")
+		(lib_id "Okapi-eagle-import:3V3_AUX")
 		(at 68.58 50.8 0)
 		(unit 1)
@@
 			)
 		)
-		(property "Value" "VCC"
+		(property "Value" "3V3_AUX"
 			(at 66.04 53.34 90)
 			(show_name no)
@@
 	)
 	(symbol
-		(lib_id "Okapi-eagle-import:supply1_371_VCC")
+		(lib_id "Okapi-eagle-import:3V3_AUX")
 		(at 43.18 58.42 0)
 		(unit 1)
@@
 			)
 		)
-		(property "Value" "VCC"
+		(property "Value" "3V3_AUX"
 			(at 40.64 60.96 90)
 			(show_name no)
@@
 	)
 	(symbol
-		(lib_id "Okapi-eagle-import:supply1_371_VCC")
+		(lib_id "Okapi-eagle-import:3V3_AUX")
 		(at 60.96 96.52 0)
 		(unit 1)
@@
 			)
 		)
-		(property "Value" "VCC"
+		(property "Value" "3V3_AUX"
 			(at 58.42 99.06 90)
 			(show_name no)
@@
 	)
 	(symbol
-		(lib_id "Okapi-eagle-import:supply1_371_VCC")
+		(lib_id "Okapi-eagle-import:3V3_AUX")
 		(at 68.58 109.22 0)
 		(unit 1)
@@
 			)
 		)
-		(property "Value" "VCC"
+		(property "Value" "3V3_AUX"
 			(at 66.04 111.76 90)
 			(show_name no)
@@
 	)
 	(symbol
-		(lib_id "Okapi-eagle-import:supply1_371_VCC")
+		(lib_id "Okapi-eagle-import:3V3_CORE")
 		(at 182.88 175.26 0)
 		(unit 1)
@@
 			)
 		)
-		(property "Value" "VCC"
+		(property "Value" "3V3_CORE"
 			(at 180.34 177.8 90)
 			(show_name no)
@@
 	)
 	(symbol
-		(lib_id "Okapi-eagle-import:supply1_371_VCC")
+		(lib_id "Okapi-eagle-import:3V3_AUX")
 		(at 22.86 60.96 0)
 		(unit 1)
@@
 			)
 		)
-		(property "Value" "VCC"
+		(property "Value" "3V3_AUX"
 			(at 20.32 63.5 90)
 			(show_name no)
@@
 	)
 	(symbol
-		(lib_id "Okapi-eagle-import:supply1_371_VCC")
+		(lib_id "Okapi-eagle-import:3V3_AUX")
 		(at 22.86 119.38 0)
 		(unit 1)
@@
 			)
 		)
-		(property "Value" "VCC"
+		(property "Value" "3V3_AUX"
 			(at 20.32 121.92 90)
 			(show_name no)
@@
 	)
 	(symbol
-		(lib_id "Okapi-eagle-import:supply1_371_VCC")
+		(lib_id "Okapi-eagle-import:3V3_AUX")
 		(at 60.96 38.1 0)
 		(unit 1)
@@
 			)
 		)
-		(property "Value" "VCC"
+		(property "Value" "3V3_AUX"
 			(at 58.42 40.64 90)
 			(show_name no)
@@
 	)
 	(symbol
-		(lib_id "Okapi-eagle-import:supply1_371_VCC")
+		(lib_id "Okapi-eagle-import:3V3_AUX")
 		(at 43.18 116.84 0)
 		(unit 1)
@@
 			)
 		)
-		(property "Value" "VCC"
+		(property "Value" "3V3_AUX"
 			(at 40.64 119.38 90)
 			(show_name no)
