File: Hardware/KiCAD-10import/Okapi_5.kicad_sch (KiCad schematic)
At the start: 29 parts, among them U30 MCP4726SOT-23, U31 BME280, U32 PAC1934QFN, U33 ADS111, U38 MLX90393, U43 BMA456, U44 VEML6030

Commit message: KiCAD-10import: fix power net and label errors from Eagle import
- Okapi_2: P+1-4,6-9 → 3V3_AUX; P+5,P+10 → 3V3_CORE (were all VCC)
- Okapi_3: SUPPLY9,SUPPLY10 → 3V3_CORE (were VCC)
- Okapi_5: P+11 → 3V3_AUX (was VCC)
- Okapi_2: QOD global labels → FEATHER_BAT (Eagle net name)
- Okapi root: add V_CORE net label on U6-OUT/U9-VIN/C17/C43 wire

The Eagle→KiCad importer assigns all P+/SUPPLY power symbols the
generic "VCC" net regardless of the actual net they sit on in Eagle.
The correct rail assignments were traced from the Eagle netlist.

Co-Authored-By: Claude Sonnet 4.6 <noreply@anthropic.com>
Connections:
- net VCC is gone; now on net 3V3_AUX: U31.2 (CSB), U31.6 (VDDIO), U31.8 (VDD)
Changed lines of the file:
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@@
 	)
 	(symbol
-		(lib_id "Okapi-eagle-import:supply1_371_VCC")
+		(lib_id "Okapi-eagle-import:3V3_AUX")
 		(at 124.46 101.6 0)
 		(unit 1)
@@
 			)
 		)
-		(property "Value" "VCC"
+		(property "Value" "3V3_AUX"
 			(at 121.92 104.14 90)
 			(show_name no)
