File: Hardware/KiCAD-10import/Okapi_3.kicad_sch (KiCad schematic)
At the start: 56 parts, among them J1 CONN_82.54_SCREW, J2 CONN_102.54_SCREW, J3 CONN_42.54_SCREW, J4 CONN_82.54_SCREW, J5 CONN_022.54_SCREW, J6 CONN_022.54_SCREW, J7 CONN_022.54_SCREW, J8 JST_2MM_MALE, J9 B_SERIES_M.2EKEY_NOPROG, Q4 2N7002, U35 MB85RC, U45 PCA9634QFN

Commit message: KiCAD-10import: fix power net and label errors from Eagle import
- Okapi_2: P+1-4,6-9 → 3V3_AUX; P+5,P+10 → 3V3_CORE (were all VCC)
- Okapi_3: SUPPLY9,SUPPLY10 → 3V3_CORE (were VCC)
- Okapi_5: P+11 → 3V3_AUX (was VCC)
- Okapi_2: QOD global labels → FEATHER_BAT (Eagle net name)
- Okapi root: add V_CORE net label on U6-OUT/U9-VIN/C17/C43 wire

The Eagle→KiCad importer assigns all P+/SUPPLY power symbols the
generic "VCC" net regardless of the actual net they sit on in Eagle.
The correct rail assignments were traced from the Eagle netlist.

Co-Authored-By: Claude Sonnet 4.6 <noreply@anthropic.com>
Connections:
- net VCC is gone; now on net 3V3_CORE: D5.2 (ANODE), R45.2
Changed lines of the file:
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@@
 	)
 	(symbol
-		(lib_id "Okapi-eagle-import:VCC")
+		(lib_id "Okapi-eagle-import:3V3_CORE")
 		(at 220.98 254 0)
 		(unit 1)
@@
 			)
 		)
-		(property "Value" "VCC"
+		(property "Value" "3V3_CORE"
 			(at 220.98 251.206 0)
 			(show_name no)
@@
 	)
 	(symbol
-		(lib_id "Okapi-eagle-import:VCC")
+		(lib_id "Okapi-eagle-import:3V3_CORE")
 		(at 271.78 261.62 0)
 		(unit 1)
@@
 			)
 		)
-		(property "Value" "VCC"
+		(property "Value" "3V3_CORE"
 			(at 271.78 258.826 0)
 			(show_name no)

Commit message: KiCAD-10import: mark B-Series SIM and UB_USB pins as no-connect
All four external SIM interface pins (SIM_VCC, SIM_CLK, SIM_DATA,
SIM_RST) and the UB USB interface pins (UB_VBUS, UB_USB_N, UB_USB_P)
are intentionally unconnected: the B-Series uses its onboard eSIM
and the secondary USB-to-modem interface is not needed.

Removes the stray global labels that the KiCad importer created
from these unconnected pins, and replaces them with proper
no-connect markers on J9.

Co-Authored-By: Claude Sonnet 4.6 <noreply@anthropic.com>
Connections:
- net 3V3_CORE: no longer R18.2, R53.2, R60.2, R64.2, R76.2, R77.2, R78.2, R79.2, R80.2, U35.8 (VDD), U45.20 (A1), U45.3 (A4)
- net 3V3_FEATHER: no longer R86.2
- net FEATHER_CTS: no longer MS1.20 (GPIO6)
- net FEATHER_GPIO: no longer MS1.10 (GPIOA5)
- net FEATHER_RTS: no longer MS1.19 (GPIO5)
- net GND: no longer J2.10, J9.1 (GND@1), J9.15 (GND@15), J9.3 (GND@3), J9.49 (AGND@49), J9.5 (GND@5), J9.56 (GND@56), J9.7 (GND@7), J9.76 (GND@76), J9.9 (GND@9), J9.GND (GND@1), MS1.4 (GND), U45.14 (A5), U45.19 (A0)
- net LI+: no longer J6.P2 (2)
- net MISO: no longer J9.50 (MISO)
- net MOSI_BUF: no longer J9.52 (MOSI), MS1.12 (GPIOMOSI)
- net SCK_BUF: no longer MS1.11 (GPIOSCK)
- net SCL: no longer U35.6 (SCL)
- net SCL_FEATHER: no longer MS1.18 (GPIOSCL)
- net SDA_FEATHER: no longer J9.22 (SDA)
- net SDA_OB: no longer U35.5 (SDA), U45.17 (SDA)
- net TX: no longer MS1.14 (GPIORX)
- net VBUS_PRIME: no longer J1.2
- net VBUS_SEC: no longer J4.2
- net WD_DONE: no longer MS1.8 (GPIOA3)
- net 3V3_AUX: no longer names the net of SD1.4 (VDD)
- net 3V3_AUX: no longer R41.2
- net 5V_AUX: no longer names the net of F2.2
- net 5V_AUX: no longer MS1.26 (USB)
- net CS_OUT: no longer names the net of J2.6
- net DAC_OUT: no longer names the net of J1.7
- net FEATHER_BAT: no longer names the net of J9.2 (VCC@2), J9.4 (VCC@4), J9.6 (VCC@6), J9.8 (VCC@8)
- net FEATHER_BAT: no longer MS1.28 (VBAT)
- net GPIO_1_OUT: no longer names the net of J1.5
- net GPIO_2_OUT: no longer names the net of J4.7
- net GPIO_3_OUT: no longer names the net of J4.8
- net LED1: no longer names the net of R44.1
- net LED2: no longer names the net of R42.1
- net LI-: no longer names the net of J6.P1 (1)
- net LI-: no longer J8.1 (-)
- net LOG_INT: no longer names the net of R45.1, S3.3 (4), S3.4 (3)
- net RST: no longer names the net of Q4.3 (D)
- net RST: no longer ISP1.5 (RST)
- net RX: no longer names the net of J9.36 (TX)
- net RX: no longer MS1.15 (GPIOTX)
- net SCK_OUT: no longer names the net of J2.3
- net SCL_OUT_PRIME: no longer names the net of J2.7
- net SCL_OUT_SEC: no longer names the net of J4.4
- net SDA_OUT_SEC: no longer names the net of J4.3
- net SIM_VCC: no longer names the net of J9.67 (SIM_VCC)
- net UB_VBUS: no longer names the net of J9.74 (UB_VBUS)
- net V_PRIME: no longer names the net of R73.2
- net V_PRIME_SENSE: no longer names the net of J5.P2 (2), R73.1
- net V_SOLAR: no longer names the net of J7.P2 (2)
- new net: R53.2, R60.2, R64.2, R76.2, R77.2, R78.2, R79.2, R80.2
- new net: J9.1 (GND@1), J9.3 (GND@3), J9.5 (GND@5), J9.7 (GND@7), J9.9 (GND@9), J9.GND (GND@1)
- no-connect marks 0 -> 7
